Commit message: made URDF

File: URDF Robot v4/URDF_description/target.urdf (robot description, URDF)
Before this commit: robot URDF, 15 links, 14 joints
Links:
- removed link Component103_1
- removed link Component104_1
- removed link old_component__14__1
- removed link old_component__15__1
- removed link old_component__16__1
- removed link old_component__17__1
- removed link old_component__18__1
- removed link old_component__19__1
- removed link old_component__20__1
- removed link old_component__21__1
- removed link old_component__22__1
- removed link old_component__23__1
- removed link old_component__24__1
- removed link old_component__25__1
- added link l1_1, mass 0.260658112795213; collision mesh filename=package://URDF_description/meshes/l1_1.stl scale=0.001 0.001 0.001; visual mesh filename=package://URDF_description/meshes/l1_1.stl scale=0.001 0.001 0.001
- added link l2_1, mass 0.2606766909017712; collision mesh filename=package://URDF_description/meshes/l2_1.stl scale=0.001 0.001 0.001; visual mesh filename=package://URDF_description/meshes/l2_1.stl scale=0.001 0.001 0.001
- added link l3_1, mass 0.2605710862815951; collision mesh filename=package://URDF_description/meshes/l3_1.stl scale=0.001 0.001 0.001; visual mesh filename=package://URDF_description/meshes/l3_1.stl scale=0.001 0.001 0.001
- added link l4_1, mass 0.4795683297989441; collision mesh filename=package://URDF_description/meshes/l4_1.stl scale=0.001 0.001 0.001; visual mesh filename=package://URDF_description/meshes/l4_1.stl scale=0.001 0.001 0.001
- added link l5_1, mass 0.5723786894338777; collision mesh filename=package://URDF_description/meshes/l5_1.stl scale=0.001 0.001 0.001; visual mesh filename=package://URDF_description/meshes/l5_1.stl scale=0.001 0.001 0.001
- added link l6_1, mass 0.260583085238151; collision mesh filename=package://URDF_description/meshes/l6_1.stl scale=0.001 0.001 0.001; visual mesh filename=package://URDF_description/meshes/l6_1.stl scale=0.001 0.001 0.001
- added link l7_1, mass 0.42535185084301863; collision mesh filename=package://URDF_description/meshes/l7_1.stl scale=0.001 0.001 0.001; visual mesh filename=package://URDF_description/meshes/l7_1.stl scale=0.001 0.001 0.001
- added link r1_1, mass 0.260645951134301; collision mesh filename=package://URDF_description/meshes/r1_1.stl scale=0.001 0.001 0.001; visual mesh filename=package://URDF_description/meshes/r1_1.stl scale=0.001 0.001 0.001
- added link r2_1, mass 0.2606418768017664; collision mesh filename=package://URDF_description/meshes/r2_1.stl scale=0.001 0.001 0.001; visual mesh filename=package://URDF_description/meshes/r2_1.stl scale=0.001 0.001 0.001
- added link r3_1, mass 0.26058347817133687; collision mesh filename=package://URDF_description/meshes/r3_1.stl scale=0.001 0.001 0.001; visual mesh filename=package://URDF_description/meshes/r3_1.stl scale=0.001 0.001 0.001
- added link r4_1, mass 0.4795660415586759; collision mesh filename=package://URDF_description/meshes/r4_1.stl scale=0.001 0.001 0.001; visual mesh filename=package://URDF_description/meshes/r4_1.stl scale=0.001 0.001 0.001
- added link r5_1, mass 0.5723780660401575; collision mesh filename=package://URDF_description/meshes/r5_1.stl scale=0.001 0.001 0.001; visual mesh filename=package://URDF_description/meshes/r5_1.stl scale=0.001 0.001 0.001
- added link r6_1, mass 0.26058568857338693; collision mesh filename=package://URDF_description/meshes/r6_1.stl scale=0.001 0.001 0.001; visual mesh filename=package://URDF_description/meshes/r6_1.stl scale=0.001 0.001 0.001
- added link r7_1, mass 0.42535393165731183; collision mesh filename=package://URDF_description/meshes/r7_1.stl scale=0.001 0.001 0.001; visual mesh filename=package://URDF_description/meshes/r7_1.stl scale=0.001 0.001 0.001
Joints:
- joint Revolute 46: child old_component__25__1 -> l3_1; parent old_component__24__1 -> l2_1
- joint Revolute 54: child old_component__23__1 -> r3_1; parent old_component__15__1 -> r2_1
- joint Revolute 66: child old_component__20__1 -> l4_1; parent old_component__25__1 -> l3_1
- joint Revolute 67: child old_component__19__1 -> l5_1; parent old_component__20__1 -> l4_1
- joint Revolute 68: child old_component__22__1 -> l6_1; parent old_component__19__1 -> l5_1
- joint Revolute 69: child old_component__21__1 -> l7_1; parent old_component__22__1 -> l6_1
- joint Revolute 70: child old_component__17__1 -> r4_1; parent old_component__23__1 -> r3_1
- joint Revolute 71: child old_component__16__1 -> r5_1; parent old_component__17__1 -> r4_1
- joint Revolute 72: child old_component__14__1 -> r6_1; parent old_component__16__1 -> r5_1
- joint Revolute 73: child old_component__18__1 -> r7_1; parent old_component__14__1 -> r6_1
- joint Revolute 90: child Component104_1 -> r1_1
- joint Revolute 91: child Component103_1 -> l1_1
- joint Revolute 92: child old_component__24__1 -> l2_1; parent Component103_1 -> l1_1
- joint Revolute 93: child old_component__15__1 -> r2_1; parent Component104_1 -> r1_1
