Commit message: fixed missing meshes issue

File: URDF Robot v4/URDF_description/urdf/URDF.xacro (robot description, xacro)
@@ -24,5 +24,5 @@
   </collision>
 </link>
-<link name="old_component__25__1">
+<link name="l3_1">
   <inertial>
     <origin xyz="-0.0010554319034483655 -0.010177955025813722 0.0099605153071331" rpy="0 0 0"/>
@@ -33,5 +33,5 @@
     <origin xyz="0.01125 0.056859 -0.300753" rpy="0 0 0"/>
     <geometry>
-      <mesh filename="package://URDF_description/meshes/old_component__25__1.stl" scale="0.001 0.001 0.001"/>
+      <mesh filename="package://URDF_description/meshes/l3_1.stl" scale="0.001 0.001 0.001"/>
     </geometry>
     <material name="silver"/>
@@ -40,9 +40,9 @@
     <origin xyz="0.01125 0.056859 -0.300753" rpy="0 0 0"/>
     <geometry>
-      <mesh filename="package://URDF_description/meshes/old_component__25__1.stl" scale="0.001 0.001 0.001"/>
-    </geometry>
-  </collision>
-</link>
-<link name="old_component__23__1">
+      <mesh filename="package://URDF_description/meshes/l3_1.stl" scale="0.001 0.001 0.001"/>
+    </geometry>
+  </collision>
+</link>
+<link name="r3_1">
   <inertial>
     <origin xyz="-0.0013721079730043672 0.010183257082741967 0.009960041415219167" rpy="0 0 0"/>
@@ -53,5 +53,5 @@
     <origin xyz="0.010932 -0.07264 -0.300746" rpy="0 0 0"/>
     <geometry>
-      <mesh filename="package://URDF_description/meshes/old_component__23__1.stl" scale="0.001 0.001 0.001"/>
+      <mesh filename="package://URDF_description/meshes/r3_1.stl" scale="0.001 0.001 0.001"/>
     </geometry>
     <material name="silver"/>
@@ -60,9 +60,9 @@
     <origin xyz="0.010932 -0.07264 -0.300746" rpy="0 0 0"/>
     <geometry>
-      <mesh filename="package://URDF_description/meshes/old_component__23__1.stl" scale="0.001 0.001 0.001"/>
-    </geometry>
-  </collision>
-</link>
-<link name="old_component__20__1">
+      <mesh filename="package://URDF_description/meshes/r3_1.stl" scale="0.001 0.001 0.001"/>
+    </geometry>
+  </collision>
+</link>
+<link name="l4_1">
   <inertial>
     <origin xyz="-0.025108010465582926 0.020534482343403035 -0.07938553469074466" rpy="0 0 0"/>
@@ -73,5 +73,5 @@
     <origin xyz="-0.015754 0.067037 -0.300753" rpy="0 0 0"/>
     <geometry>
-      <mesh filename="package://URDF_description/meshes/old_component__20__1.stl" scale="0.001 0.001 0.001"/>
+      <mesh filename="package://URDF_description/meshes/l4_1.stl" scale="0.001 0.001 0.001"/>
     </geometry>
     <material name="silver"/>
@@ -80,9 +80,9 @@
     <origin xyz="-0.015754 0.067037 -0.300753" rpy="0 0 0"/>
     <geometry>
-      <mesh filename="package://URDF_description/meshes/old_component__20__1.stl" scale="0.001 0.001 0.001"/>
-    </geometry>
-  </collision>
-</link>
-<link name="old_component__19__1">
+      <mesh filename="package://URDF_description/meshes/l4_1.stl" scale="0.001 0.001 0.001"/>
+    </geometry>
+  </collision>
+</link>
+<link name="l5_1">
   <inertial>
     <origin xyz="-0.029491082579912755 0.0039567541577458926 -0.1016008471361324" rpy="0 0 0"/>
@@ -93,5 +93,5 @@
     <origin xyz="0.009024 0.071577 -0.195159" rpy="0 0 0"/>
     <geometry>
-      <mesh filename="package://URDF_description/meshes/old_component__19__1.stl" scale="0.001 0.001 0.001"/>
+      <mesh filename="package://URDF_description/meshes/l5_1.stl" scale="0.001 0.001 0.001"/>
     </geometry>
     <material name="silver"/>
@@ -100,9 +100,9 @@
     <origin xyz="0.009024 0.071577 -0.195159" rpy="0 0 0"/>
     <geometry>
-      <mesh filename="package://URDF_description/meshes/old_component__19__1.stl" scale="0.001 0.001 0.001"/>
-    </geometry>
-  </collision>
-</link>
-<link name="old_component__22__1">
+      <mesh filename="package://URDF_description/meshes/l5_1.stl" scale="0.001 0.001 0.001"/>
+    </geometry>
+  </collision>
+</link>
+<link name="l6_1">
   <inertial>
     <origin xyz="0.010148909868078046 0.0014454123231728566 0.009960061611517447" rpy="0 0 0"/>
@@ -113,5 +113,5 @@
     <origin xyz="0.018503 0.067568 -0.050454" rpy="0 0 0"/>
     <geometry>
-      <mesh filename="package://URDF_description/meshes/old_component__22__1.stl" scale="0.001 0.001 0.001"/>
+      <mesh filename="package://URDF_description/meshes/l6_1.stl" scale="0.001 0.001 0.001"/>
     </geometry>
     <material name="silver"/>
@@ -120,9 +120,9 @@
     <origin xyz="0.018503 0.067568 -0.050454" rpy="0 0 0"/>
     <geometry>
-      <mesh filename="package://URDF_description/meshes/old_component__22__1.stl" scale="0.001 0.001 0.001"/>
-    </geometry>
-  </collision>
-</link>
-<link name="old_component__21__1">
+      <mesh filename="package://URDF_description/meshes/l6_1.stl" scale="0.001 0.001 0.001"/>
+    </geometry>
+  </collision>
+</link>
+<link name="l7_1">
   <inertial>
     <origin xyz="-0.0038360250370360807 0.0260878632088187 -0.050533848086451186" rpy="0 0 0"/>
@@ -133,5 +133,5 @@
     <origin xyz="0.008354 0.094498 -0.050454" rpy="0 0 0"/>
     <geometry>
-      <mesh filename="package://URDF_description/meshes/old_component__21__1.stl" scale="0.001 0.001 0.001"/>
+      <mesh filename="package://URDF_description/meshes/l7_1.stl" scale="0.001 0.001 0.001"/>
     </geometry>
     <material name="silver"/>
@@ -140,9 +140,9 @@
     <origin xyz="0.008354 0.094498 -0.050454" rpy="0 0 0"/>
     <geometry>
-      <mesh filename="package://URDF_description/meshes/old_component__21__1.stl" scale="0.001 0.001 0.001"/>
-    </geometry>
-  </collision>
-</link>
-<link name="old_component__17__1">
+      <mesh filename="package://URDF_description/meshes/l7_1.stl" scale="0.001 0.001 0.001"/>
+    </geometry>
+  </collision>
+</link>
+<link name="r4_1">
   <inertial>
     <origin xyz="-0.025086134509350884 -0.019584458432278365 -0.07938591030825276" rpy="0 0 0"/>
@@ -153,5 +153,5 @@
     <origin xyz="-0.016072 -0.082823 -0.300746" rpy="0 0 0"/>
     <geometry>
-      <mesh filename="package://URDF_description/meshes/old_component__17__1.stl" scale="0.001 0.001 0.001"/>
+      <mesh filename="package://URDF_description/meshes/r4_1.stl" scale="0.001 0.001 0.001"/>
     </geometry>
     <material name="silver"/>
@@ -160,9 +160,9 @@
     <origin xyz="-0.016072 -0.082823 -0.300746" rpy="0 0 0"/>
     <geometry>
-      <mesh filename="package://URDF_description/meshes/old_component__17__1.stl" scale="0.001 0.001 0.001"/>
-    </geometry>
-  </collision>
-</link>
-<link name="old_component__16__1">
+      <mesh filename="package://URDF_description/meshes/r4_1.stl" scale="0.001 0.001 0.001"/>
+    </geometry>
+  </collision>
+</link>
+<link name="r5_1">
   <inertial>
     <origin xyz="-0.029491076838213486 -0.003956632577475125 -0.10160079326267875" rpy="0 0 0"/>
@@ -173,5 +173,5 @@
     <origin xyz="0.008684 -0.088313 -0.195152" rpy="0 0 0"/>
     <geometry>
-      <mesh filename="package://URDF_description/meshes/old_component__16__1.stl" scale="0.001 0.001 0.001"/>
+      <mesh filename="package://URDF_description/meshes/r5_1.stl" scale="0.001 0.001 0.001"/>
     </geometry>
     <material name="silver"/>
@@ -180,9 +180,9 @@
     <origin xyz="0.008684 -0.088313 -0.195152" rpy="0 0 0"/>
     <geometry>
-      <mesh filename="package://URDF_description/meshes/old_component__16__1.stl" scale="0.001 0.001 0.001"/>
-    </geometry>
-  </collision>
-</link>
-<link name="old_component__14__1">
+      <mesh filename="package://URDF_description/meshes/r5_1.stl" scale="0.001 0.001 0.001"/>
+    </geometry>
+  </collision>
+</link>
+<link name="r6_1">
   <inertial>
     <origin xyz="0.010216801636088587 -0.0014452836669609503 0.009959962708194117" rpy="0 0 0"/>
@@ -193,5 +193,5 @@
     <origin xyz="0.018163 -0.084304 -0.050447" rpy="0 0 0"/>
     <geometry>
-      <mesh filename="package://URDF_description/meshes/old_component__14__1.stl" scale="0.001 0.001 0.001"/>
+      <mesh filename="package://URDF_description/meshes/r6_1.stl" scale="0.001 0.001 0.001"/>
     </geometry>
     <material name="silver"/>
@@ -200,9 +200,9 @@
     <origin xyz="0.018163 -0.084304 -0.050447" rpy="0 0 0"/>
     <geometry>
-      <mesh filename="package://URDF_description/meshes/old_component__14__1.stl" scale="0.001 0.001 0.001"/>
-    </geometry>
-  </collision>
-</link>
-<link name="old_component__18__1">
+      <mesh filename="package://URDF_description/meshes/r6_1.stl" scale="0.001 0.001 0.001"/>
+    </geometry>
+  </collision>
+</link>
+<link name="r7_1">
   <inertial>
     <origin xyz="-0.003836011886673152 -0.025999620351597932 -0.050533600876661144" rpy="0 0 0"/>
@@ -213,5 +213,5 @@
     <origin xyz="0.007946 -0.111234 -0.050447" rpy="0 0 0"/>
     <geometry>
-      <mesh filename="package://URDF_description/meshes/old_component__18__1.stl" scale="0.001 0.001 0.001"/>
+      <mesh filename="package://URDF_description/meshes/r7_1.stl" scale="0.001 0.001 0.001"/>
     </geometry>
     <material name="silver"/>
@@ -220,9 +220,9 @@
     <origin xyz="0.007946 -0.111234 -0.050447" rpy="0 0 0"/>
     <geometry>
-      <mesh filename="package://URDF_description/meshes/old_component__18__1.stl" scale="0.001 0.001 0.001"/>
-    </geometry>
-  </collision>
-</link>
-<link name="Component104_1">
+      <mesh filename="package://URDF_description/meshes/r7_1.stl" scale="0.001 0.001 0.001"/>
+    </geometry>
+  </collision>
+</link>
+<link name="r1_1">
   <inertial>
     <origin xyz="0.0004996878831269973 0.02734500634448242 0.00896780014474241" rpy="0 0 0"/>
@@ -233,5 +233,5 @@
     <origin xyz="0.011804 -0.008368 -0.332395" rpy="0 0 0"/>
     <geometry>
-      <mesh filename="package://URDF_description/meshes/Component104_1.stl" scale="0.001 0.001 0.001"/>
+      <mesh filename="package://URDF_description/meshes/r1_1.stl" scale="0.001 0.001 0.001"/>
     </geometry>
     <material name="silver"/>
@@ -240,9 +240,9 @@
     <origin xyz="0.011804 -0.008368 -0.332395" rpy="0 0 0"/>
     <geometry>
-      <mesh filename="package://URDF_description/meshes/Component104_1.stl" scale="0.001 0.001 0.001"/>
-    </geometry>
-  </collision>
-</link>
-<link name="Component103_1">
+      <mesh filename="package://URDF_description/meshes/r1_1.stl" scale="0.001 0.001 0.001"/>
+    </geometry>
+  </collision>
+</link>
+<link name="l1_1">
   <inertial>
     <origin xyz="0.0001816438125570169 -0.0273436447861984 0.008967326406254417" rpy="0 0 0"/>
@@ -253,5 +253,5 @@
     <origin xyz="0.011804 -0.008368 -0.332395" rpy="0 0 0"/>
     <geometry>
-      <mesh filename="package://URDF_description/meshes/Component103_1.stl" scale="0.001 0.001 0.001"/>
+      <mesh filename="package://URDF_description/meshes/l1_1.stl" scale="0.001 0.001 0.001"/>
     </geometry>
     <material name="silver"/>
@@ -260,9 +260,9 @@
     <origin xyz="0.011804 -0.008368 -0.332395" rpy="0 0 0"/>
     <geometry>
-      <mesh filename="package://URDF_description/meshes/Component103_1.stl" scale="0.001 0.001 0.001"/>
-    </geometry>
-  </collision>
-</link>
-<link name="old_component__24__1">
+      <mesh filename="package://URDF_description/meshes/l1_1.stl" scale="0.001 0.001 0.001"/>
+    </geometry>
+  </collision>
+</link>
+<link name="l2_1">
   <inertial>
     <origin xyz="-0.009584482225170093 0.002892011357412988 -0.010242130854528853" rpy="0 0 0"/>
@@ -273,5 +273,5 @@
     <origin xyz="0.011622 0.028932 -0.310995" rpy="0 0 0"/>
     <geometry>
-      <mesh filename="package://URDF_description/meshes/old_component__24__1.stl" scale="0.001 0.001 0.001"/>
+      <mesh filename="package://URDF_description/meshes/l2_1.stl" scale="0.001 0.001 0.001"/>
     </geometry>
     <material name="silver"/>
@@ -280,9 +280,9 @@
     <origin xyz="0.011622 0.028932 -0.310995" rpy="0 0 0"/>
     <geometry>
-      <mesh filename="package://URDF_description/meshes/old_component__24__1.stl" scale="0.001 0.001 0.001"/>
-    </geometry>
-  </collision>
-</link>
-<link name="old_component__15__1">
+      <mesh filename="package://URDF_description/meshes/l2_1.stl" scale="0.001 0.001 0.001"/>
+    </geometry>
+  </collision>
+</link>
+<link name="r2_1">
   <inertial>
     <origin xyz="-0.00958582114085108 -0.0028961550072031106 -0.010249054751743758" rpy="0 0 0"/>
@@ -293,5 +293,5 @@
     <origin xyz="0.011304 -0.045668 -0.310995" rpy="0 0 0"/>
     <geometry>
-      <mesh filename="package://URDF_description/meshes/old_component__15__1.stl" scale="0.001 0.001 0.001"/>
+      <mesh filename="package://URDF_description/meshes/r2_1.stl" scale="0.001 0.001 0.001"/>
     </geometry>
     <material name="silver"/>
@@ -300,5 +300,5 @@
     <origin xyz="0.011304 -0.045668 -0.310995" rpy="0 0 0"/>
     <geometry>
-      <mesh filename="package://URDF_description/meshes/old_component__15__1.stl" scale="0.001 0.001 0.001"/>
+      <mesh filename="package://URDF_description/meshes/r2_1.stl" scale="0.001 0.001 0.001"/>
     </geometry>
   </collision>
@@ -306,60 +306,60 @@
 <joint name="Revolute 46" type="continuous">
   <origin xyz="0.000372 -0.027927 -0.010242" rpy="0 0 0"/>
-  <parent link="old_component__24__1"/>
-  <child link="old_component__25__1"/>
+  <parent link="l2_1"/>
+  <child link="l3_1"/>
   <axis xyz="-0.0 -1.0 -0.0"/>
 </joint>
 <joint name="Revolute 54" type="continuous">
   <origin xyz="0.000372 0.026972 -0.010249" rpy="0 0 0"/>
-  <parent link="old_component__15__1"/>
-  <child link="old_component__23__1"/>
+  <parent link="r2_1"/>
+  <child link="r3_1"/>
   <axis xyz="-0.0 1.0 0.0"/>
 </joint>
 <joint name="Revolute 66" type="continuous">
   <origin xyz="0.027004 -0.010178 0.0" rpy="0 0 0"/>
-  <parent link="old_component__25__1"/>
-  <child link="old_component__20__1"/>
+  <parent link="l3_1"/>
+  <child link="l4_1"/>
   <axis xyz="1.0 0.0 -0.0"/>
 </joint>
 <joint name="Revolute 67" type="continuous">
   <origin xyz="-0.024778 -0.00454 -0.105594" rpy="0 0 0"/>
-  <parent link="old_component__20__1"/>
-  <child link="old_component__19__1"/>
+  <parent link="l4_1"/>
+  <child link="l5_1"/>
   <axis xyz="-0.0 -1.0 -0.0"/>
 </joint>
 <joint name="Revolute 68" type="continuous">
   <origin xyz="-0.009479 0.004009 -0.144705" rpy="0 0 0"/>
-  <parent link="old_component__19__1"/>
-  <child link="old_component__22__1"/>
+  <parent link="l5_1"/>
+  <child link="l6_1"/>
   <axis xyz="1.0 0.0 0.0"/>
 </joint>
 <joint name="Revolute 69" type="continuous">
   <origin xyz="0.010149 -0.02693 0.0" rpy="0 0 0"/>
-  <parent link="old_component__22__1"/>
-  <child link="old_component__21__1"/>
+  <parent link="l6_1"/>
+  <child link="l7_1"/>
   <axis xyz="0.0 -1.0 -0.0"/>
 </joint>
 <joint name="Revolute 70" type="continuous">
   <origin xyz="0.027004 0.010183 0.0" rpy="0 0 0"/>
-  <parent link="old_component__23__1"/>
-  <child link="old_component__17__1"/>
+  <parent link="r3_1"/>
+  <child link="r4_1"/>
   <axis xyz="1.0 0.0 -0.0"/>
 </joint>
 <joint name="Revolute 71" type="continuous">
   <origin xyz="-0.024756 0.00549 -0.105594" rpy="0 0 0"/>
-  <parent link="old_component__17__1"/>
-  <child link="old_component__16__1"/>
+  <parent link="r4_1"/>
+  <child link="r5_1"/>
   <axis xyz="-0.0 1.0 0.0"/>
 </joint>
 <joint name="Revolute 72" type="continuous">
   <origin xyz="-0.009479 -0.004009 -0.144705" rpy="0 0 0"/>
-  <parent link="old_component__16__1"/>
-  <child link="old_component__14__1"/>
+  <parent link="r5_1"/>
+  <child link="r6_1"/>
   <axis xyz="1.0 0.0 -0.0"/>
 </joint>
 <joint name="Revolute 73" type="continuous">
   <origin xyz="0.010217 0.02693 0.0" rpy="0 0 0"/>
-  <parent link="old_component__14__1"/>
-  <child link="old_component__18__1"/>
+  <parent link="r6_1"/>
+  <child link="r7_1"/>
   <axis xyz="-0.0 1.0 0.0"/>
 </joint>
@@ -367,5 +367,5 @@
   <origin xyz="-0.011804 0.008368 0.332395" rpy="0 0 0"/>
   <parent link="base_link"/>
-  <child link="Component104_1"/>
+  <child link="r1_1"/>
   <axis xyz="0.0 -0.0 1.0"/>
 </joint>
@@ -373,17 +373,17 @@
   <origin xyz="-0.011804 0.008368 0.332395" rpy="0 0 0"/>
   <parent link="base_link"/>
-  <child link="Component103_1"/>
+  <child link="l1_1"/>
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